File: MakerPlayground_Sensor_ALS-PT19-315C_v1/MakerPlayground_Sensor_ALS-PT19-315C_v1.sch (KiCad schematic (older format))
At the start: 3 parts, among them J1 Conn_01x04, Q1 Q_Photo_NPN_CE

Commit message: Fix MP Light sensor mounting hole & connector.
Parts:
- J1: footprint Connector_JST:JST_PH_S4B-PH-K_1x04_P2.00mm_Horizontal -> Connector_JST:JST_PH_S4B-PH-SM4-TB_1x04-1MP_P2.00mm_Horizontal
Changed lines of the file:
@@
 EESchema Schematic File Version 4
-LIBS:MakerPlayground_ALS-PT19-315C-cache
 EELAYER 26 0
 EELAYER END
@@
 F 0 "J1" H 5700 3850 50  0000 C CNN
 F 1 "Conn_01x04" H 5850 3950 50  0000 C CNN
-F 2 "Connector_JST:JST_PH_S4B-PH-K_1x04_P2.00mm_Horizontal" H 5550 3950 50  0001 C CNN
+F 2 "Connector_JST:JST_PH_S4B-PH-SM4-TB_1x04-1MP_P2.00mm_Horizontal" H 5550 3950 50  0001 C CNN
 F 3 "~" H 5550 3950 50  0001 C CNN
 	1    5550 3950
