File: MakerPlayground_Sensor_PushButton_v1/MakerPlayground_Sensor_PushButton_v1.sch (KiCad schematic (older format))
At the start: 3 parts, among them J1 Connector, SW1 SW_DPST_x2

Commit message: Add mounting hole & change to SMD connector.
Parts:
- J1: footprint Connector_JST:JST_PH_S4B-PH-K_1x04_P2.00mm_Horizontal -> Connector_JST:JST_PH_S4B-PH-SM4-TB_1x04-1MP_P2.00mm_Horizontal
Changed lines of the file:
@@
 EESchema Schematic File Version 4
-LIBS:Button-cache
 EELAYER 26 0
 EELAYER END
@@
 F 0 "J1" H 6830 3192 50  0000 L CNN
 F 1 "Connector" H 6830 3101 50  0000 L CNN
-F 2 "Connector_JST:JST_PH_S4B-PH-K_1x04_P2.00mm_Horizontal" H 6750 3200 50  0001 C CNN
+F 2 "Connector_JST:JST_PH_S4B-PH-SM4-TB_1x04-1MP_P2.00mm_Horizontal" H 6750 3200 50  0001 C CNN
 F 3 "~" H 6750 3200 50  0001 C CNN
 	1    6750 3200
