File: MakerPlayground_Sensor_Temperature_Humidity_SHT3X_v1/MakerPlayground_Sensor_Temperature_Humidity_SHT3X_v1.sch (KiCad schematic (older format))
At the start: 5 parts, among them J1 Conn_01x04, U1 Sensirion_SHT3x

Commit message: Add mounting hole & change to SMD connector.
Parts:
- J1: footprint Connector_JST:JST_PH_S4B-PH-K_1x04_P2.00mm_Horizontal -> Connector_JST:JST_PH_S4B-PH-SM4-TB_1x04-1MP_P2.00mm_Horizontal
Changed lines of the file:
@@
 EESchema Schematic File Version 4
-LIBS:SHT3x-cache
 EELAYER 26 0
 EELAYER END
@@
 F 0 "J1" H 7130 3892 50  0000 L CNN
 F 1 "Conn_01x04" H 7130 3801 50  0000 L CNN
-F 2 "Connector_JST:JST_PH_S4B-PH-K_1x04_P2.00mm_Horizontal" H 7050 3900 50  0001 C CNN
+F 2 "Connector_JST:JST_PH_S4B-PH-SM4-TB_1x04-1MP_P2.00mm_Horizontal" H 7050 3900 50  0001 C CNN
 F 3 "~" H 7050 3900 50  0001 C CNN
 	1    7050 3900
