File: MakerPlayground_Sensor_Temperature_Humidity_SHT3X_v1/MakerPlayground_Sensor_Temperature_Humidity_SHT3X_v1.kicad_pcb (KiCad board)
At the start: 2 copper layers, 30.4 x 19.9 mm, 8 parts, among them J1 Conn_01x04, U1 Sensirion_SHT3x

Commit message: Complete design.
Other:
- board text added: "v1.0"
Changed lines of the file:
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@@
   (general
     (thickness 1.6)
-    (drawings 223)
+    (drawings 224)
     (tracks 50)
     (zones 0)
@@
       (xy 0.199355 -0.596628) (xy 0.593328 -0.992663) (xy 0.790777 -0.991434)) (layer F.SilkS) (width 0.01))
   )
+  (gr_text v1.0 (at 140.25 114) (layer F.SilkS)
+    (effects (font (size 0.5 0.5) (thickness 0.1)))
+  )
   (gr_line (start 124 107.743) (end 126.5 107.743) (layer Edge.Cuts) (width 0.1))
