File: MakerPlayground_Actuator_PiezoBuzzer_v1/MakerPlayground_Actuator_PiezoBuzzer_v1.kicad_pcb (KiCad board)
At the start: 2 copper layers, 22.5 x 19.9 mm, 4 parts, among them J1 Conn_01x04

Commit message: Design complete.
Parts:
- added REF**: MountingHole_3mm, MountingHole:MountingHole_3mm, F.Cu at (116.5, 100.0)
- added REF**: MountingHole_3mm, MountingHole:MountingHole_3mm, F.Cu at (146.5, 100.0)
Other:
- board size 22.5 x 19.9 mm -> 35.5 x 19.9 mm
- board text added: "v1.0"
