File: MakerPlayground_Actuator_H-BridgeMotorDriver_v1/MakerPlayground_HbridgeMotorDriver.kicad_pcb (KiCad board)
At the start: 2 copper layers, 45.5 x 32 mm, 16 parts, among them J1 Conn_01x04, J2 Screw_Terminal_01x02, J3 Screw_Terminal_01x02, U1 ROHM_BD62110AEFJ

Commit message: Complete design.
Other:
- board text added: "v1.0"
Changed lines of the file:
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@@
   (general
     (thickness 1.6)
-    (drawings 302)
+    (drawings 303)
     (tracks 89)
     (zones 0)
@@
     (pad 1 np_thru_hole circle (at 0 0) (size 3 3) (drill 3) (layers *.Cu *.Mask))
   )
+  (gr_text v1.0 (at 157.5 74.5 90) (layer F.SilkS)
+    (effects (font (size 0.5 0.5) (thickness 0.1)))
+  )
   (gr_line (start 152.597 64.5676) (end 152.52 64.5583) (layer Edge.Cuts) (width 0.1))
