File: MakerPlayground_Actuator_RGB-LED_SK9822_v1/MakerPlayground_Actuator_RGB-LED_SK9822_v1.kicad_pcb (KiCad board)
At the start: 2 copper layers, 30.4 x 19.9 mm, 6 parts, among them J1 Conn_01x04

Commit message: Design complete.
Other:
- board text added: "v1.0"
Changed lines of the file:
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@@
   (general
     (thickness 1.6)
-    (drawings 223)
+    (drawings 224)
     (tracks 33)
     (zones 0)
@@
     (pad 1 np_thru_hole circle (at 0 0) (size 3 3) (drill 3) (layers *.Cu *.Mask))
   )
+  (gr_text v1.0 (at 140.25 109) (layer F.SilkS)
+    (effects (font (size 0.5 0.5) (thickness 0.1)))
+  )
   (gr_line (start 149 102.7) (end 146.4 102.7) (layer Edge.Cuts) (width 0.15))
