File: MakerPlayground_Sensor_BD1020HPV_v1/MakerPlayground_Sensor_BD1020HPV_v1.kicad_pcb (KiCad board)
At the start: 2 copper layers, 30.4 x 19.9 mm, 6 parts, among them J1 Conn_01x04, U1 BD1020HFV

Commit message: Complete design.
Other:
- board text added: "v1.0"
Changed lines of the file:
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@@
   (general
     (thickness 1.6)
-    (drawings 223)
+    (drawings 224)
     (tracks 17)
     (zones 0)
@@
     (pad 1 np_thru_hole circle (at 0 0) (size 3 3) (drill 3) (layers *.Cu *.Mask))
   )
+  (gr_text v1.0 (at 140.25 113.5) (layer F.SilkS)
+    (effects (font (size 0.5 0.5) (thickness 0.1)))
+  )
   (gr_line (start 141.819 95.1136) (end 141.739 95.0916) (layer Edge.Cuts) (width 0.1))
