File: MakerPlayground_Actuator_SSD1306_OLEDv1/MakerPlayground_Actuator_SSD1306_OLEDv1.kicad_pcb (KiCad board)
At the start: 2 copper layers, 28 x 28 mm, 6 parts, among them J1 OLED_CONN, J2 JST_CONN

Commit message: Doing to job ngai. Still not complete jaaa.
Parts:
- added REF**: MountingHole_3mm, MountingHole:MountingHole_3mm, F.Cu at (115.0, 105.0)
- added REF**: MountingHole_3mm, MountingHole:MountingHole_3mm, F.Cu at (92.0, 105.0)
- added REF**: MountingHole_3mm, MountingHole:MountingHole_3mm, F.Cu at (115.0, 82.0)
- added REF**: MountingHole_3mm, MountingHole:MountingHole_3mm, F.Cu at (92.0, 82.0)
- moved J1 0.48 mm to (99.7, 81.0)
- moved J2 0.25 mm to (106.5, 101.0)
Routing:
- added copper zone on B.Cu, net GND
- added copper zone on F.Cu, net GND

Commit message: Complete
Parts:
- removed C1: 1uF, Capacitor_SMD:C_0603_1608Metric
- removed C2: 0.1uF, Capacitor_SMD:C_0603_1608Metric
- removed R1, R2: 10K, Resistor_SMD:R_0603_1608Metric
- removed the REF** at (115.0, 105.0)
- removed the REF** at (92.0, 105.0)
- removed the REF** at (115.0, 82.0)
- removed the REF** at (92.0, 82.0)
- added G***: LOGO, GiraffeTech-Utility:MakerPlayground_logo_2x2mm, B.Cu at (103.5, 92.2)
- added REF**: MountingHole_4mm, MountingHole:MountingHole_4mm, F.Cu at (92.2, 104.8)
- added REF**: MountingHole_4mm, MountingHole:MountingHole_4mm, F.Cu at (114.8, 104.8)
- added REF**: MountingHole_4mm, MountingHole:MountingHole_4mm, F.Cu at (114.8, 82.2)
- added REF**: MountingHole_4mm, MountingHole:MountingHole_4mm, F.Cu at (92.2, 82.2)
Connections:
- J1 pad 3: SDA -> SCL
- J1 pad 4: SCL -> SDA
Routing:
- net VCC: track 0.00 -> 33.2 mm
- net SDA: track 0.00 -> 22.0 mm
- net SCL: track 0.00 -> 21.8 mm
Other:
- board text added: "OLED Screen"
