File: MakerPlayground_Actuator_SSD1306_OLEDv1/MakerPlayground_Actuator_SSD1306_OLEDv1.sch (KiCad schematic (older format))
At the start: 6 parts, among them J1 OLED_CONN, J2 JST_CONN

Commit message: Complete
Parts:
- removed C1: 1uF, Capacitor_SMD:C_0603_1608Metric, symbol Device:C_Small
- removed C2: 0.1uF, Capacitor_SMD:C_0603_1608Metric, symbol Device:C_Small
- removed R1, R2: 10K, Resistor_SMD:R_0603_1608Metric, symbol Device:R_Small
Connections:
- net SCL: now also J1.3 (Pin_3); no longer J1.4 (Pin_4)
- net SDA: now also J1.4 (Pin_4); no longer J1.3 (Pin_3)
Changed lines of the file:
@@
 EESchema Schematic File Version 4
+LIBS:MakerPlayground_Actuator_SSD1306_OLEDv1-cache
 EELAYER 26 0
 EELAYER END
@@
 Wire Wire Line
 	3900 2550 3900 2650
-Text GLabel 4000 2350 2    50   Input ~ 0
+Text GLabel 4000 2250 2    50   Input ~ 0
 SDA
 Wire Wire Line
 	3800 2350 4000 2350
-Text GLabel 4000 2250 2    50   Input ~ 0
+Text GLabel 4000 2350 2    50   Input ~ 0
 SCL
 Wire Wire Line
@@
 Wire Wire Line
 	4350 2450 4350 2150
-$Comp
-L Device:R_Small R1
-U 1 1 5CADA020
-P 4850 2350
-F 0 "R1" H 4909 2396 50  0000 L CNN
-F 1 "10K" H 4909 2305 50  0000 L CNN
-F 2 "Resistor_SMD:R_0603_1608Metric" H 4850 2350 50  0001 C CNN
-F 3 "~" H 4850 2350 50  0001 C CNN
-	1    4850 2350
-	1    0    0    -1
-$EndComp
-$Comp
-L power:VCC #PWR0105
-U 1 1 5CADA0CC
-P 4850 2150
-F 0 "#PWR0105" H 4850 2000 50  0001 C CNN
-F 1 "VCC" H 4867 2323 50  0000 C CNN
-F 2 "" H 4850 2150 50  0001 C CNN
-F 3 "" H 4850 2150 50  0001 C CNN
-	1    4850 2150
-	1    0    0    -1
-$EndComp
-$Comp
-L Device:R_Small R2
-U 1 1 5CADA0F8
-P 5250 2350
-F 0 "R2" H 5309 2396 50  0000 L CNN
-F 1 "10K" H 5309 2305 50  0000 L CNN
-F 2 "Resistor_SMD:R_0603_1608Metric" H 5250 2350 50  0001 C CNN
-F 3 "~" H 5250 2350 50  0001 C CNN
-	1    5250 2350
-	1    0    0    -1
-$EndComp
-$Comp
-L power:VCC #PWR0106
-U 1 1 5CADA0FE
-P 5250 2150
-F 0 "#PWR0106" H 5250 2000 50  0001 C CNN
-F 1 "VCC" H 5267 2323 50  0000 C CNN
-F 2 "" H 5250 2150 50  0001 C CNN
-F 3 "" H 5250 2150 50  0001 C CNN
-	1    5250 2150
-	1    0    0    -1
-$EndComp
-Wire Wire Line
-	4850 2150 4850 2250
-Wire Wire Line
-	5250 2150 5250 2250
-Wire Wire Line
-	4850 2450 4850 2550
-Wire Wire Line
-	5250 2450 5250 2550
-Text GLabel 4850 2550 3    50   Input ~ 0
-SDA
-Text GLabel 5250 2550 3    50   Input ~ 0
-SCL
-$Comp
-L power:VCC #PWR0107
-U 1 1 5CADA93C
-P 5900 2150
-F 0 "#PWR0107" H 5900 2000 50  0001 C CNN
-F 1 "VCC" H 5917 2323 50  0000 C CNN
-F 2 "" H 5900 2150 50  0001 C CNN
-F 3 "" H 5900 2150 50  0001 C CNN
-	1    5900 2150
-	1    0    0    -1
-$EndComp
-Wire Wire Line
-	5900 2150 5900 2250
-$Comp
-L Device:C_Small C1
-U 1 1 5CADAAB9
-P 5900 2350
-F 0 "C1" H 5992 2396 50  0000 L CNN
-F 1 "1uF" H 5992 2305 50  0000 L CNN
-F 2 "Capacitor_SMD:C_0603_1608Metric" H 5900 2350 50  0001 C CNN
-F 3 "~" H 5900 2350 50  0001 C CNN
-	1    5900 2350
-	1    0    0    -1
-$EndComp
-$Comp
-L power:VCC #PWR0108
-U 1 1 5CADAB42
-P 6300 2150
-F 0 "#PWR0108" H 6300 2000 50  0001 C CNN
-F 1 "VCC" H 6317 2323 50  0000 C CNN
-F 2 "" H 6300 2150 50  0001 C CNN
-F 3 "" H 6300 2150 50  0001 C CNN
-	1    6300 2150
-	1    0    0    -1
-$EndComp
-Wire Wire Line
-	6300 2150 6300 2250
-$Comp
-L Device:C_Small C2
-U 1 1 5CADAB49
-P 6300 2350
-F 0 "C2" H 6392 2396 50  0000 L CNN
-F 1 "0.1uF" H 6392 2305 50  0000 L CNN
-F 2 "Capacitor_SMD:C_0603_1608Metric" H 6300 2350 50  0001 C CNN
-F 3 "~" H 6300 2350 50  0001 C CNN
-	1    6300 2350
-	1    0    0    -1
-$EndComp
-$Comp
-L power:GND #PWR0109
-U 1 1 5CADAE91
-P 5900 2550
-F 0 "#PWR0109" H 5900 2300 50  0001 C CNN
-F 1 "GND" H 5905 2377 50  0000 C CNN
-F 2 "" H 5900 2550 50  0001 C CNN
-F 3 "" H 5900 2550 50  0001 C CNN
-	1    5900 2550
-	1    0    0    -1
-$EndComp
-$Comp
-L power:GND #PWR0110
-U 1 1 5CADAEAF
-P 6300 2550
-F 0 "#PWR0110" H 6300 2300 50  0001 C CNN
-F 1 "GND" H 6305 2377 50  0000 C CNN
-F 2 "" H 6300 2550 50  0001 C CNN
-F 3 "" H 6300 2550 50  0001 C CNN
-	1    6300 2550
-	1    0    0    -1
-$EndComp
-Wire Wire Line
-	6300 2450 6300 2550
-Wire Wire Line
-	5900 2450 5900 2550
 $EndSCHEMATC
