File: MakerPlayground_Sensor_LIS3DH_v1/MakerPlayground_Sensor_LIS3DH_v1.kicad_pcb (KiCad board)
At the start: 2 copper layers, 30.4 x 19.9 mm, 17 parts, among them J1 Conn_01x04, Q1 BSS138, Q2 BSS138, U1 AP2127K-3.3, U2 LIS3DH

Commit message: Single HEX design; Lock mounting hole footprint & review mounting hole position.
Routing:
- net GND: vias 16 -> 10
Changed lines of the file:
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@@
     (thickness 1.6)
     (drawings 238)
-    (tracks 153)
+    (tracks 147)
     (zones 0)
     (modules 17)
@@
     (add_net VCC)
   )
-  (module MountingHole:MountingHole_3mm (layer F.Cu)
+  (module MountingHole:MountingHole_3mm locked (layer F.Cu)
     (at 159 100)
     (descr "Mounting Hole 3mm, no annular")
@@
     )
   )
-  (module MountingHole:MountingHole_3mm (layer F.Cu)
+  (module MountingHole:MountingHole_3mm locked (layer F.Cu)
     (at 134 100)
     (descr "Mounting Hole 3mm, no annular")
@@
   (segment (start 146.5 100.75) (end 146.5 99.75) (width 0.25) (layer F.Cu) (net 2))
   (via (at 148.75 102.5) (size 0.6) (drill 0.3) (layers F.Cu B.Cu) (net 2))
-  (via (at 140.25 106.5) (size 0.6) (drill 0.3) (layers F.Cu B.Cu) (net 2))
-  (via (at 142.75 106.5) (size 0.6) (drill 0.3) (layers F.Cu B.Cu) (net 2))
   (via (at 145.25 106.5) (size 0.6) (drill 0.3) (layers F.Cu B.Cu) (net 2))
   (via (at 147.75 106.5) (size 0.6) (drill 0.3) (layers F.Cu B.Cu) (net 2))
-  (via (at 150.25 106.5) (size 0.6) (drill 0.3) (layers F.Cu B.Cu) (net 2))
-  (via (at 152.75 106.5) (size 0.6) (drill 0.3) (layers F.Cu B.Cu) (net 2))
-  (via (at 147.75 91) (size 0.6) (drill 0.3) (layers F.Cu B.Cu) (net 2))
-  (via (at 145.25 91) (size 0.6) (drill 0.3) (layers F.Cu B.Cu) (net 2))
   (via (at 142.75 91) (size 0.6) (drill 0.3) (layers F.Cu B.Cu) (net 2))
   (via (at 150.25 91) (size 0.6) (drill 0.3) (layers F.Cu B.Cu) (net 2))

Commit message: Complete design.
Other:
- board text added: "v1.0"
Changed lines of the file:
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@@
   (general
     (thickness 1.6)
-    (drawings 238)
+    (drawings 239)
     (tracks 147)
     (zones 0)
@@
     (pad 1 np_thru_hole circle (at 0 0) (size 3 3) (drill 3) (layers *.Cu *.Mask))
   )
+  (gr_text v1.0 (at 151 109) (layer F.SilkS)
+    (effects (font (size 0.5 0.5) (thickness 0.1)))
+  )
   (gr_line (start 149.9 90.0387) (end 149.395 90.0387) (layer Edge.Cuts) (width 0.1))

Commit message: Fix missing capacitor description. Complete.
Parts:
- removed G***: LOGO, GiraffeTech-Utility:MakerPlayground_logo_2x2mm
- C4: value CP1 -> 22uF
- R5: value 10k -> 10K
Connections:
- U1 pad 4: (no net) -> Net-(U1-Pad4)
- U2 pad 11: (no net) -> Net-(U2-Pad11)
- U2 pad 13: (no net) -> Net-(U2-Pad13)
- U2 pad 15: (no net) -> Net-(U2-Pad15)
- U2 pad 16: (no net) -> Net-(U2-Pad16)
- U2 pad 2: (no net) -> Net-(U2-Pad2)
- U2 pad 3: (no net) -> Net-(U2-Pad3)
- U2 pad 9: (no net) -> Net-(U2-Pad9)
Changed lines of the file:
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@@
     (tracks 147)
     (zones 0)
-    (modules 17)
-    (nets 9)
+    (modules 16)
+    (nets 17)
   )
   (page A4)
@@
   (net 7 SCL_3V3)
   (net 8 "Net-(R5-Pad1)")
+  (net 9 "Net-(U1-Pad4)")
+  (net 10 "Net-(U2-Pad9)")
+  (net 11 "Net-(U2-Pad11)")
+  (net 12 "Net-(U2-Pad13)")
+  (net 13 "Net-(U2-Pad3)")
+  (net 14 "Net-(U2-Pad2)")
+  (net 15 "Net-(U2-Pad16)")
+  (net 16 "Net-(U2-Pad15)")
   (net_class Default "This is the default net class."
     (clearance 0.2)
@@
     (add_net GND)
     (add_net "Net-(R5-Pad1)")
+    (add_net "Net-(U1-Pad4)")
+    (add_net "Net-(U2-Pad11)")
+    (add_net "Net-(U2-Pad13)")
+    (add_net "Net-(U2-Pad15)")
+    (add_net "Net-(U2-Pad16)")
+    (add_net "Net-(U2-Pad2)")
+    (add_net "Net-(U2-Pad3)")
+    (add_net "Net-(U2-Pad9)")
     (add_net SCL_3V3)
     (add_net SCL_VIN)
@@
     (fp_line (start 1.5 1.5) (end -1.5 1.5) (layer F.SilkS) (width 0.15))
     (fp_line (start -1.5 1.5) (end -1.5 -1.1) (layer F.SilkS) (width 0.15))
-    (pad 9 smd rect (at 1.225 1) (size 0.35 0.25) (layers F.Cu F.Paste F.Mask))
+    (pad 9 smd rect (at 1.225 1) (size 0.35 0.25) (layers F.Cu F.Paste F.Mask)
+      (net 10 "Net-(U2-Pad9)"))
     (pad 10 smd rect (at 1.225 0.5) (size 0.35 0.25) (layers F.Cu F.Paste F.Mask)
       (net 2 GND))
-    (pad 11 smd rect (at 1.225 0) (size 0.35 0.25) (layers F.Cu F.Paste F.Mask))
+    (pad 11 smd rect (at 1.225 0) (size 0.35 0.25) (layers F.Cu F.Paste F.Mask)
+      (net 11 "Net-(U2-Pad11)"))
     (pad 12 smd rect (at 1.225 -0.5) (size 0.35 0.25) (layers F.Cu F.Paste F.Mask)
       (net 2 GND))
-    (pad 13 smd rect (at 1.225 -1) (size 0.35 0.25) (layers F.Cu F.Paste F.Mask))
+    (pad 13 smd rect (at 1.225 -1) (size 0.35 0.25) (layers F.Cu F.Paste F.Mask)
+      (net 12 "Net-(U2-Pad13)"))
     (pad 5 smd rect (at -1.225 1) (size 0.35 0.25) (layers F.Cu F.Paste F.Mask)
       (net 2 GND))
     (pad 4 smd rect (at -1.225 0.5) (size 0.35 0.25) (layers F.Cu F.Paste F.Mask)
       (net 7 SCL_3V3))
-    (pad 3 smd rect (at -1.225 0) (size 0.35 0.25) (layers F.Cu F.Paste F.Mask))
-    (pad 2 smd rect (at -1.225 -0.5) (size 0.35 0.25) (layers F.Cu F.Paste F.Mask))
+    (pad 3 smd rect (at -1.225 0) (size 0.35 0.25) (layers F.Cu F.Paste F.Mask)
+      (net 13 "Net-(U2-Pad3)"))
+    (pad 2 smd rect (at -1.225 -0.5) (size 0.35 0.25) (layers F.Cu F.Paste F.Mask)
+      (net 14 "Net-(U2-Pad2)"))
     (pad 1 smd rect (at -1.225 -1) (size 0.35 0.25) (layers F.Cu F.Paste F.Mask)
       (net 3 +3V3))
-    (pad 16 smd rect (at -0.5 -1.275) (size 0.25 0.35) (layers F.Cu F.Paste F.Mask))
-    (pad 15 smd rect (at 0 -1.275) (size 0.25 0.35) (layers F.Cu F.Paste F.Mask))
+    (pad 16 smd rect (at -0.5 -1.275) (size 0.25 0.35) (layers F.Cu F.Paste F.Mask)
+      (net 15 "Net-(U2-Pad16)"))
+    (pad 15 smd rect (at 0 -1.275) (size 0.25 0.35) (layers F.Cu F.Paste F.Mask)
+      (net 16 "Net-(U2-Pad15)"))
     (pad 14 smd rect (at 0.5 -1.275) (size 0.25 0.35) (layers F.Cu F.Paste F.Mask)
       (net 3 +3V3))
@@
       (effects (font (size 1 1) (thickness 0.15)))
     )
-    (fp_text value CP1 (at 0 1.75) (layer F.Fab)
+    (fp_text value 22uF (at 0 1.75) (layer F.Fab)
       (effects (font (size 1 1) (thickness 0.15)))
     )
@@
     (pad 3 smd rect (at -1.1 0.95 270) (size 1.06 0.65) (layers F.Cu F.Paste F.Mask)
       (net 1 VCC))
-    (pad 4 smd rect (at 1.1 0.95 270) (size 1.06 0.65) (layers F.Cu F.Paste F.Mask))
+    (pad 4 smd rect (at 1.1 0.95 270) (size 1.06 0.65) (layers F.Cu F.Paste F.Mask)
+      (net 9 "Net-(U1-Pad4)"))
     (pad 5 smd rect (at 1.1 -0.95 270) (size 1.06 0.65) (layers F.Cu F.Paste F.Mask)
       (net 3 +3V3))
@@
       (effects (font (size 1 1) (thickness 0.15)))
     )
-    (fp_text value 10k (at 0 1.65 270) (layer F.Fab)
+    (fp_text value 10K (at 0 1.65 270) (layer F.Fab)
       (effects (font (size 1 1) (thickness 0.15)))
     )
@@
     )
   )
-  (module GiraffeTech-Utility:MakerPlayground_logo_2x2mm (layer F.Cu)
-    (at 146.5 92.5)
-    (fp_text reference G*** (at 0 0) (layer F.SilkS) hide
-      (effects (font (size 1.524 1.524) (thickness 0.3)))
-    )
-    (fp_text value LOGO (at 0.75 0) (layer F.SilkS) hide
-      (effects (font (size 1.524 1.524) (thickness 0.3)))
-    )
-    (fp_poly (pts (xy 0.992188 -0.564543) (xy 0.992164 -0.528929) (xy 0.992097 -0.495895) (xy 0.991991 -0.466261)
-      (xy 0.991852 -0.440843) (xy 0.991684 -0.420459) (xy 0.991492 -0.405926) (xy 0.991282 -0.398062)
-      (xy 0.99116 -0.396875) (xy 0.988207 -0.399571) (xy 0.980351 -0.407199) (xy 0.968291 -0.419067)
-      (xy 0.952725 -0.434484) (xy 0.934354 -0.452758) (xy 0.913876 -0.4732) (xy 0.906847 -0.480231)
-      (xy 0.823563 -0.563586) (xy 0.907875 -0.647899) (xy 0.992188 -0.732211) (xy 0.992188 -0.564543)) (layer F.SilkS) (width 0.01))
-    (fp_poly (pts (xy 0.992272 -0.049513) (xy 0.991238 0.124084) (xy 0.990203 0.297682) (xy 0.731231 0.038685)
-      (xy 0.472259 -0.220311) (xy 0.559597 -0.307581) (xy 0.646934 -0.394851) (xy 0.992272 -0.049513)) (layer F.SilkS) (width 0.01))
-    (fp_poly (pts (xy 0.306845 -0.036934) (xy 0.315366 -0.028902) (xy 0.328804 -0.015931) (xy 0.346812 0.001638)
-      (xy 0.369045 0.023463) (xy 0.39516 0.049204) (xy 0.424812 0.078521) (xy 0.457655 0.111071)
-      (xy 0.493344 0.146515) (xy 0.531535 0.184511) (xy 0.571883 0.224719) (xy 0.614044 0.266798)
-      (xy 0.649934 0.302669) (xy 0.992273 0.645025) (xy 0.990203 0.990203) (xy 0.559594 0.560703)
-      (xy 0.128984 0.131202) (xy 0.214278 0.045757) (xy 0.235683 0.024442) (xy 0.255382 0.005068)
-      (xy 0.272657 -0.011676) (xy 0.28679 -0.025103) (xy 0.297063 -0.034528) (xy 0.302757 -0.039261)
-      (xy 0.303583 -0.039687) (xy 0.306845 -0.036934)) (layer F.SilkS) (width 0.01))
-    (fp_poly (pts (xy 0.790777 -0.991434) (xy 0.988227 -0.990203) (xy -0.992187 0.990197) (xy -0.992187 -0.992187)
-      (xy -0.601395 -0.992187) (xy -0.646963 -0.945555) (xy -0.665935 -0.926151) (xy -0.688266 -0.903332)
-      (xy -0.711752 -0.879346) (xy -0.734194 -0.856442) (xy -0.745114 -0.845303) (xy -0.797697 -0.791685)
-      (xy -0.698482 -0.692529) (xy -0.599266 -0.593373) (xy -0.399829 -0.79278) (xy -0.200393 -0.992187)
-      (xy 0.195473 -0.992187) (xy -0.099139 -0.695955) (xy -0.39375 -0.399723) (xy -0.194618 -0.200591)
-      (xy 0.199355 -0.596628) (xy 0.593328 -0.992663) (xy 0.790777 -0.991434)) (layer F.SilkS) (width 0.01))
-  )
   (module Connector_JST:JST_PH_S4B-PH-SM4-TB_1x04-1MP_P2.00mm_Horizontal (layer B.Cu)
